File: 93ng-blue-aux/93ng-blue-aux-esp32-only.sch (KiCad schematic (older format))
At the start: 24 parts, among them J1 12V INPUT, J2 ESP32 UART, J3 ESP32 JTAG, J7 I-BUS, SW1 SW_DIP_x01, U1 ESP32-WROOM-32D, U2 BA33DD0T, U3 MC33897

Commit message: More work on standalone ESP32 module
Parts:
- removed J3: ESP32 JTAG, Connector_PinHeader_2.54mm:PinHeader_1x04_P2.54mm_Vertical, symbol Connector:Conn_01x04_Male
- removed R2: 100, Resistor_SMD:R_0805_2012Metric_Pad1.15x1.40mm_HandSolder, symbol Device:R_Small
- removed SW1: SW_DIP_x01, Button_Switch_SMD:SW_DIP_SPSTx01_Slide_Omron_A6S-110x_W8.9mm_P2.54mm, symbol Switch:SW_DIP_x01
- removed U2: BA33DD0T, Package_TO_SOT_THT:TO-220-3_Vertical, symbol custom_symbols:BA33DD0T
- added C3: 1nF, Capacitor_SMD:C_0805_2012Metric_Pad1.15x1.40mm_HandSolder, symbol Device:C_Small
- added C6, C7, C8: 10uF, Capacitor_SMD:C_0805_2012Metric_Pad1.15x1.40mm_HandSolder, symbol Device:C_Small
- added D2: PWR_LED, LED_SMD:LED_0805_2012Metric_Pad1.15x1.40mm_HandSolder, symbol Device:LED
- added D4: 1N5819, Diode_THT:D_DO-41_SOD81_P10.16mm_Horizontal, symbol Diode:1N5819
- added J3: USB_C_Receptacle_USB2.0, Connector_USB:USB_C_Receptacle_Amphenol_12401610E4-2A, symbol Connector:USB_C_Receptacle_USB2.0
- added Q1, Q2: S8050, Package_TO_SOT_SMD:SOT-23_Handsoldering, symbol Transistor_BJT:S8050
- added R11: 1K, Resistor_SMD:R_0805_2012Metric_Pad1.15x1.40mm_HandSolder, symbol Device:R_Small
- added R12: 470, Resistor_SMD:R_0805_2012Metric_Pad1.15x1.40mm_HandSolder, symbol Device:R_Small
- added R2: 2k, Resistor_SMD:R_0805_2012Metric_Pad1.15x1.40mm_HandSolder, symbol Device:R
- added R8: 12K, Resistor_SMD:R_0805_2012Metric_Pad1.15x1.40mm_HandSolder, symbol Device:R_Small
- added SW1: PWR IN SELECT, Connector_PinHeader_2.54mm:PinHeader_1x03_P2.54mm_Vertical, symbol Switch:SW_SPDT
- added U2: NCP1117-3.3_SOT223, Package_TO_SOT_SMD:SOT-223-3_TabPin2, symbol Regulator_Linear:NCP1117-3.3_SOT223
- added U4: FUSB302BMPX, Package_DFN_QFN:WQFN-14-1EP_2.5x2.5mm_P0.5mm_EP1.45x1.45mm, symbol Interface_USB:FUSB302BMPX
- added U5: CP2102N-A01-GQFN28, Package_DFN_QFN:QFN-28-1EP_5x5mm_P0.5mm_EP3.35x3.35mm, symbol Interface_USB:CP2102N-A01-GQFN28
- C2: value 0.1uF -> 10uF
- R1: value 1k -> 12K
- R3, R4: value 100 -> 5k
- R5: value 100 -> 12K
Connections:
- net labels added: DTR, ESP32_BOOT, ESP32_EN, ESP32_RX, ESP32_TX, FUSB_INTN, FUSB_SCL, FUSB_SDA, RTS, USB_CC1, USB_CC2, USB_D+, USB_D-, USB_VBUS
- net labels removed: ESP32_BOOTOPT
- wire segments 65 -> 67
Other:
- note added: "12V TO 3.3V LDO\n1A OUTPUT"
- note added: "ESP32 \nAUTO-BOOTMODE\nSELECTOR\nTHINGY"
- note added: "USB TYPE C PORT"
- note added: "USB-UART INTERFACE"
- note added: "USB3.1 PD CONTROLLER"
- note removed: "12V TO 3.3V\n2A OUTPUT"
- note removed: "SYSTEM CONFIG SWITCHES\nUSED TO PUT ESP32 OR BM62\nINTO PROGRAM MODE"
- moved on the sheet: C1, C2, C4, C5, D1, D3, J1, J2, J7, L1, R10, R6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

Commit message: Placed all the components roughly! Added ground plane!
Parts:
- C1: footprint Capacitor_THT:CP_Radial_D10.0mm_P5.00mm -> Capacitor_SMD:C_2010_5025Metric_Pad1.52x2.65mm_HandSolder
- D4: footprint Diode_THT:D_DO-41_SOD81_P10.16mm_Horizontal -> Diode_SMD:D_0805_2012Metric_Pad1.15x1.40mm_HandSolder
- J3: manf# (none) -> 12401610E4#2A
- Q1, Q2: manf# (none) -> MMS8050-H-TP
- U1: manf# (none) -> ESP32-WROOM-32D
- U4: manf# (none) -> FUSB302BMPX
- U5: manf# (none) -> CP2102N-A02-GQFN24
Changed lines of the file:
@@
 F 2 "RF_Module:ESP32-WROOM-32" H 2150 3100 50  0001 C CNN
 F 3 "https://www.espressif.com/sites/default/files/documentation/esp32-wroom-32d_esp32-wroom-32u_datasheet_en.pdf" H 1850 4650 50  0001 C CNN
+F 4 "ESP32-WROOM-32D" H 2150 4600 50  0001 C CNN "manf#"
 	1    2150 4600
 	1    0    0    -1
@@
 F 2 "Package_DFN_QFN:QFN-28-1EP_5x5mm_P0.5mm_EP3.35x3.35mm" H 8200 1750 50  0001 L CNN
 F 3 "https://www.silabs.com/documents/public/data-sheets/cp2102n-datasheet.pdf" H 7800 2200 50  0001 C CNN
+F 4 "CP2102N-A02-GQFN24" V 7750 2950 50  0001 C CNN "manf#"
 	1    7750 2950
 	1    0    0    -1
@@
 F 2 "Package_DFN_QFN:WQFN-14-1EP_2.5x2.5mm_P0.5mm_EP1.45x1.45mm" H 5850 3250 50  0001 C CNN
 F 3 "http://www.onsemi.com/pub/Collateral/FUSB302B-D.PDF" H 5950 3350 50  0001 C CNN
+F 4 "FUSB302BMPX" H 5850 3750 50  0001 C CNN "manf#"
 	1    5850 3750
 	1    0    0    -1
@@
 F 2 "Connector_USB:USB_C_Receptacle_Amphenol_12401610E4-2A" H 6050 2000 50  0001 C CNN
 F 3 "https://www.usb.org/sites/default/files/documents/usb_type-c.zip" H 6050 2000 50  0001 C CNN
+F 4 "12401610E4#2A" V 5900 2000 50  0001 C CNN "manf#"
 	1    5900 2000
 	0    1    1    0
@@
 F 0 "C1" H 2350 2350 50  0000 L CNN
 F 1 "10uF" H 2300 2250 50  0000 L CNN
-F 2 "Capacitor_THT:CP_Radial_D10.0mm_P5.00mm" H 2438 2150 50  0001 C CNN
+F 2 "Capacitor_SMD:C_2010_5025Metric_Pad1.52x2.65mm_HandSolder" H 2438 2150 50  0001 C CNN
 F 3 "~" H 2400 2300 50  0001 C CNN
 	1    2400 2300
@@
 F 0 "D4" V 6546 2671 50  0000 R CNN
 F 1 "1N5819" V 6455 2671 50  0000 R CNN
-F 2 "Diode_THT:D_DO-41_SOD81_P10.16mm_Horizontal" H 6500 2575 50  0001 C CNN
+F 2 "Diode_SMD:D_0805_2012Metric_Pad1.15x1.40mm_HandSolder" H 6500 2575 50  0001 C CNN
 F 3 "http://www.vishay.com/docs/88525/1n5817.pdf" H 6500 2750 50  0001 C CNN
 	1    6500 2750
@@
 F 2 "Package_TO_SOT_SMD:SOT-23_Handsoldering" H 4350 3275 50  0001 L CIN
 F 3 "http://www.unisonic.com.tw/datasheet/S8050.pdf" H 4150 3350 50  0001 L CNN
+F 4 "MMS8050-H-TP" H 4150 3350 50  0001 C CNN "manf#"
 	1    4150 3350
 	-1   0    0    1
@@
 F 2 "Package_TO_SOT_SMD:SOT-23_Handsoldering" H 4250 2425 50  0001 L CIN
 F 3 "http://www.unisonic.com.tw/datasheet/S8050.pdf" H 4050 2500 50  0001 L CNN
+F 4 "MMS8050-H-TP" H 4050 2500 50  0001 C CNN "manf#"
 	1    4050 2500
 	1    0    0    -1

Commit message: Made new version without USBC-PD chip, and simple pulldowns. Placement looks good.
Parts:
- removed U4: FUSB302BMPX, Package_DFN_QFN:WQFN-14-1EP_2.5x2.5mm_P0.5mm_EP1.45x1.45mm, symbol Interface_USB:FUSB302BMPX
- added R13, R14: 5.1k, Resistor_SMD:R_0805_2012Metric_Pad1.15x1.40mm_HandSolder, symbol Device:R_Small
Connections:
- net GND: now also R13.1, R14.1
- net USB_CC1: now also R13.2
- net USB_CC2: now also R14.2
Other:
- note added: "USB3.1 CC PULLDOWNS"
- note removed: "USB3.1 PD CONTROLLER"
Changed lines of the file:
@@
 Text GLabel 2150 6000 0    50   Input ~ 0
 GND
-$Comp
-L Connector:Conn_01x03_Male J2
-U 1 1 5E3BB7CF
-P 3350 3850
-F 0 "J2" V 3400 3550 50  0000 L CNN
-F 1 "ESP32 UART" V 3300 3550 50  0000 L CNN
-F 2 "Connector_PinHeader_2.54mm:PinHeader_1x03_P2.54mm_Vertical" H 3350 3850 50  0001 C CNN
-F 3 "~" H 3350 3850 50  0001 C CNN
-	1    3350 3850
-	-1   0    0    1
-$EndComp
 Text GLabel 3150 3750 0    50   Input ~ 0
 GND
@@
 $EndComp
 $Comp
-L Interface_USB:FUSB302BMPX U4
-U 1 1 5E52860D
-P 5850 3750
-F 0 "U4" H 5850 3261 50  0000 C CNN
-F 1 "FUSB302BMPX" H 5850 3170 50  0000 C CNN
-F 2 "Package_DFN_QFN:WQFN-14-1EP_2.5x2.5mm_P0.5mm_EP1.45x1.45mm" H 5850 3250 50  0001 C CNN
-F 3 "http://www.onsemi.com/pub/Collateral/FUSB302B-D.PDF" H 5950 3350 50  0001 C CNN
-F 4 "FUSB302BMPX" H 5850 3750 50  0001 C CNN "manf#"
-	1    5850 3750
-	1    0    0    -1
-$EndComp
-$Comp
 L Connector:USB_C_Receptacle_USB2.0 J3
 U 1 1 5E53E2D6
@@
 Text GLabel 7200 2250 0    50   Input ~ 10
 USB_VBUS
-Text GLabel 6350 3650 2    50   Input ~ 10
-USB_VBUS
 Text GLabel 6200 2600 3    50   Input ~ 10
 USB_CC2
 Text GLabel 6300 2600 3    50   Input ~ 10
 USB_CC1
-Text GLabel 6350 3750 2    50   Input ~ 10
-USB_CC1
-Text GLabel 6350 3850 2    50   Input ~ 10
-USB_CC2
 Text GLabel 5000 2000 0    50   Input ~ 0
 GND
 Text GLabel 5000 1700 0    50   Input ~ 0
-GND
-Text GLabel 5850 4150 0    50   Input ~ 0
 GND
 Text GLabel 7750 4250 0    50   Input ~ 0
@@
 Wire Wire Line
 	1600 2450 2400 2450
-Text GLabel 5750 3350 0    50   Input ~ 0
-3.3V
 Wire Wire Line
 	1700 2150 1750 2150
@@
 	0    -1   -1   0
 $EndComp
-Text GLabel 5350 3650 0    50   Input ~ 0
-FUSB_SDA
-Text GLabel 5350 3750 0    50   Input ~ 0
-FUSB_SCL
-Text GLabel 5350 3850 0    50   Input ~ 0
-FUSB_INTN
 Wire Notes Line
 	4650 3100 7100 3100
@@
 	3150 3900 3150 3950
 Text Notes 4700 3200 0    50   ~ 0
-USB3.1 PD CONTROLLER
+USB3.1 CC PULLDOWNS
 Text Notes 4700 1500 0    50   ~ 0
 USB TYPE C PORT
@@
 Wire Notes Line
 	1100 1400 8950 1400
+Text GLabel 5350 3750 0    50   Input ~ 10
+USB_CC2
+Text GLabel 5350 3650 0    50   Input ~ 10
+USB_CC1
+$Comp
+L Device:R_Small R13
+U 1 1 5E56B54F
+P 5700 3650
+F 0 "R13" V 5650 3650 50  0000 C CNN
+F 1 "5.1k" V 5600 3650 50  0000 C CNN
+F 2 "Resistor_SMD:R_0805_2012Metric_Pad1.15x1.40mm_HandSolder" H 5700 3650 50  0001 C CNN
+F 3 "~" H 5700 3650 50  0001 C CNN
+	1    5700 3650
+	0    1    1    0
+$EndComp
+$Comp
+L Device:R_Small R14
+U 1 1 5E56C633
+P 5700 3750
+F 0 "R14" V 5800 3750 50  0000 C CNN
+F 1 "5.1k" V 5850 3750 50  0000 C CNN
+F 2 "Resistor_SMD:R_0805_2012Metric_Pad1.15x1.40mm_HandSolder" H 5700 3750 50  0001 C CNN
+F 3 "~" H 5700 3750 50  0001 C CNN
+	1    5700 3750
+	0    1    1    0
+$EndComp
+Wire Wire Line
+	5350 3650 5600 3650
+Wire Wire Line
+	5600 3750 5350 3750
+Text GLabel 6050 3700 2    50   Input ~ 0
+GND
+Wire Wire Line
+	5800 3650 6050 3650
+Wire Wire Line
+	6050 3650 6050 3750
+Wire Wire Line
+	6050 3750 5800 3750
+$Comp
+L Connector:Conn_01x03_Male J2
+U 1 1 5E3BB7CF
+P 3350 3850
+F 0 "J2" V 3400 3550 50  0000 L CNN
+F 1 "ESP32 UART" V 3300 3550 50  0000 L CNN
+F 2 "Connector_PinHeader_2.54mm:PinHeader_1x03_P2.54mm_Vertical" H 3350 3850 50  0001 C CNN
+F 3 "~" H 3350 3850 50  0001 C CNN
+	1    3350 3850
+	-1   0    0    1
+$EndComp
 $EndSCHEMATC

Commit message: Updated the input power select to be an actual switch, allowing easier access if in a stacked configuration.
Parts:
- SW1: footprint Connector_PinHeader_2.54mm:PinHeader_1x03_P2.54mm_Vertical -> Button_Switch_THT:SW_E-Switch_EG1271_DPDT
Changed lines of the file:
@@
 EESchema Schematic File Version 4
-LIBS:93ng-blue-aux-esp32-only-cache
 EELAYER 30 0
 EELAYER END
@@
 F 0 "SW1" H 1950 1925 50  0000 C CNN
 F 1 "PWR IN SELECT" H 1950 2016 50  0000 C CNN
-F 2 "Connector_PinHeader_2.54mm:PinHeader_1x03_P2.54mm_Vertical" H 1950 2250 50  0001 C CNN
+F 2 "Button_Switch_THT:SW_E-Switch_EG1271_DPDT" H 1950 2250 50  0001 C CNN
 F 3 "~" H 1950 2250 50  0001 C CNN
 	1    1950 2250
