File: 93ng-blue-aux/93ng-blue-aux-esp32-interconn.kicad_pcb (KiCad board)
At the start: 2 copper layers, 50 x 50 mm, 38 parts, among them J1 12V INPUT, J2 ESP32 UART, J3 USB_C_Receptacle_USB2.0, J7 I-BUS, Q1 S8050, Q2 S8050, U1 ESP32-WROOM-32D, U2 NCP1117-3.3_SOT223, U3 MC33897, U5 CP2102N-A01-GQFN28

Commit message: Working on saab board interconnect
Parts:
- added J4: Conn_02x16_Row_Letter_First, Connector_PinHeader_1.00mm:PinHeader_2x16_P1.00mm_Vertical, F.Cu at (182.5, 82.4)
- SW1: renamed from USB <-> 12V
- moved C6 2.92 mm to (179.8, 83.2)
- moved R1 2.92 mm to (179.8, 87.5)
- moved C3 2.54 mm to (176.9, 87.5)
- moved R2 2.54 mm to (177.0, 83.2)
- moved D2 1.91 mm to (174.3, 83.2)
Routing:
- net GND: track 259.1 -> 0.00 mm
- net 3.3V: track 140.2 -> 0.00 mm
- net DTR: track 73.6 -> 0.00 mm
- net ESP32_EN: track 50.5 -> 0.00 mm, vias 2 -> 0
- net RTS: track 43.0 -> 0.00 mm, vias 2 -> 0
- net ESP32_RX: track 42.6 -> 0.00 mm, vias 1 -> 0
- net ESP32_TX: track 41.6 -> 0.00 mm, vias 1 -> 0
- net USB_VBUS: track 26.1 -> 0.00 mm, vias 1 -> 0
- net SW_CAN: track 23.0 -> 0.00 mm
- net USB_D+: track 31.8 -> 8.98 mm
- net USB_CC2: track 21.5 -> 0.00 mm
- net Net-(J1-Pad2): track 19.1 -> 0.00 mm
- net MC33_RX: track 17.8 -> 0.00 mm
- net USB_D-: track 24.6 -> 7.04 mm
- net MC33_TX: track 16.7 -> 0.00 mm, vias 2 -> 0
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
Commit message: I forget what I did.
Connections:
- C1 pad 1: Net-(C1-Pad1) -> V_IN
- J4 pad 1: (no net) -> V_IN
- J4 pad 10: (no net) -> ESP32_7
- J4 pad 11: (no net) -> ESP32_8
- J4 pad 12: (no net) -> ESP32_9
- J4 pad 13: (no net) -> ESP32_10
- J4 pad 14: (no net) -> ESP32_11
- J4 pad 15: (no net) -> ESP32_12
- J4 pad 16: (no net) -> ESP32_13
- J4 pad 17: (no net) -> ESP32_14
- J4 pad 18: (no net) -> ESP32_16
- J4 pad 19: (no net) -> ESP32_17
- J4 pad 2: (no net) -> GND
- J4 pad 20: (no net) -> ESP32_18
- J4 pad 21: (no net) -> ESP32_19
- J4 pad 22: (no net) -> ESP32_20
- J4 pad 23: (no net) -> ESP32_21
- J4 pad 24: (no net) -> ESP32_22
- J4 pad 25: (no net) -> ESP32_23
- J4 pad 26: (no net) -> ESP32_26
- J4 pad 27: (no net) -> ESP32_29
- J4 pad 28: (no net) -> ESP32_33
- J4 pad 29: (no net) -> ESP32_36
- J4 pad 3: (no net) -> 3.3V
- J4 pad 30: (no net) -> ESP32_37
- J4 pad 31: (no net) -> Net-(J4-Pad31)
- J4 pad 32: (no net) -> Net-(J4-Pad32)
- J4 pad 4: (no net) -> GND
- J4 pad 5: (no net) -> MC33_RX
- J4 pad 6: (no net) -> MC33_TX
- J4 pad 7: (no net) -> MC33_MODE0
- J4 pad 8: (no net) -> MC33_MODE1
- J4 pad 9: (no net) -> ESP32_6
- SW1 pad 2: Net-(C1-Pad1) -> V_IN
- U1 pad 10: Net-(U1-Pad10) -> ESP32_10
- U1 pad 11: Net-(U1-Pad11) -> ESP32_11
- U1 pad 12: Net-(U1-Pad12) -> ESP32_12
- U1 pad 13: Net-(U1-Pad13) -> ESP32_13
- U1 pad 14: Net-(U1-Pad14) -> ESP32_14
- U1 pad 16: Net-(U1-Pad16) -> ESP32_16
- U1 pad 17: Net-(U1-Pad17) -> ESP32_17
- U1 pad 18: Net-(U1-Pad18) -> ESP32_18
- U1 pad 19: Net-(U1-Pad19) -> ESP32_19
- U1 pad 20: Net-(U1-Pad20) -> ESP32_20
- U1 pad 21: Net-(U1-Pad21) -> ESP32_21
- U1 pad 22: Net-(U1-Pad22) -> ESP32_22
- U1 pad 23: Net-(U1-Pad23) -> ESP32_23
- U1 pad 26: Net-(U1-Pad26) -> ESP32_26
- U1 pad 29: Net-(U1-Pad29) -> ESP32_29
- U1 pad 33: Net-(U1-Pad33) -> ESP32_33
- U1 pad 36: Net-(U1-Pad36) -> ESP32_36
- U1 pad 37: Net-(U1-Pad37) -> ESP32_37
- U1 pad 6: Net-(U1-Pad6) -> ESP32_6
- U1 pad 7: Net-(U1-Pad7) -> ESP32_7
- U1 pad 8: Net-(U1-Pad8) -> ESP32_8
- U1 pad 9: Net-(U1-Pad9) -> ESP32_9
- U2 pad 3: Net-(C1-Pad1) -> V_IN
