File: 93ng-blue-aux/esp32_saab_devboard.kicad_pcb (KiCad board)
At the start: 2 copper layers, 50 x 50 mm, 28 parts, among them J1 12V INPUT, J2 ESP32 UART, J3 USB_C_Receptacle_USB2.0, J4 Conn_02x10_Counter_Clockwise, Q1 S8050, Q2 S8050, SW1 PWR IN SELECT, U1 ESP32-WROOM-32D, U2 NCP1117-3.3_SOT223, U5 CP2102N

Commit message: Switched to low-profile phoenix
Parts:
- J1: footprint TerminalBlock_Phoenix:TerminalBlock_Phoenix_MKDS-3-2-5.08_1x02_P5.08mm_Horizontal -> TerminalBlock_Phoenix:TerminalBlock_Phoenix_MKDS-1,5-2-5.08_1x02_P5.08mm_Horizontal
- U5: value CP2102N -> CP2102N-A01-GQFN28
Connections:
- J3 pad A8: (no net) -> Net-(J3-PadA8)
- J3 pad B8: (no net) -> Net-(J3-PadB8)
- U1 pad 17: (no net) -> Net-(U1-Pad17)
- U1 pad 18: (no net) -> Net-(U1-Pad18)
- U1 pad 19: (no net) -> Net-(U1-Pad19)
- U1 pad 20: (no net) -> Net-(U1-Pad20)
- U1 pad 21: (no net) -> Net-(U1-Pad21)
- U1 pad 22: (no net) -> Net-(U1-Pad22)
- U1 pad 26: (no net) -> Net-(U1-Pad26)
- U1 pad 29: (no net) -> Net-(U1-Pad29)
- U1 pad 32: (no net) -> Net-(U1-Pad32)
- U1 pad 4: (no net) -> Net-(U1-Pad4)
- U1 pad 5: (no net) -> Net-(U1-Pad5)
- U1 pad 6: (no net) -> Net-(U1-Pad6)
- U1 pad 7: (no net) -> Net-(U1-Pad7)
- U5 pad 1: (no net) -> Net-(U5-Pad1)
- U5 pad 10: (no net) -> Net-(U5-Pad10)
- U5 pad 11: (no net) -> Net-(U5-Pad11)
- U5 pad 12: (no net) -> Net-(U5-Pad12)
- U5 pad 13: (no net) -> Net-(U5-Pad13)
- U5 pad 14: (no net) -> Net-(U5-Pad14)
- U5 pad 15: (no net) -> Net-(U5-Pad15)
- U5 pad 16: (no net) -> Net-(U5-Pad16)
- U5 pad 17: (no net) -> Net-(U5-Pad17)
- U5 pad 18: (no net) -> Net-(U5-Pad18)
- U5 pad 19: (no net) -> Net-(U5-Pad19)
- U5 pad 2: (no net) -> Net-(U5-Pad2)
- U5 pad 20: (no net) -> Net-(U5-Pad20)
- U5 pad 21: (no net) -> Net-(U5-Pad21)
- U5 pad 22: (no net) -> Net-(U5-Pad22)
- U5 pad 23: (no net) -> Net-(U5-Pad23)
- U5 pad 27: (no net) -> Net-(U5-Pad27)

Commit message: Adjusted pcb text
Parts:
- U2: value NCP1117-3.3_SOT223 -> NCP1117-3.3
- U5: value CP2102N-A01-GQFN28 -> CP2102N
Changed lines of the file:
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@@
-(kicad_pcb (version 20171130) (host pcbnew 5.1.5-52549c5~84~ubuntu19.04.1)
+(kicad_pcb (version 20171130) (host pcbnew 5.1.4-e60b266~84~ubuntu19.04.1)
   (general
     (thickness 1.6)
@@
       (effects (font (size 0.5 0.5) (thickness 0.1)))
     )
-    (fp_text value CP2102N-A01-GQFN28 (at 3.628 1.016 270) (layer F.SilkS)
+    (fp_text value CP2102N (at 3.628 1.016 270) (layer F.SilkS)
       (effects (font (size 0.5 0.5) (thickness 0.1)))
     )
@@
       (effects (font (size 0.5 0.5) (thickness 0.1)))
     )
-    (fp_text value NCP1117-3.3_SOT223 (at -0.1 -0.05 180) (layer F.SilkS)
-      (effects (font (size 0.5 0.5) (thickness 0.1)))
-    )
+    (fp_text value NCP1117-3.3 (at -1.624 4 270) (layer F.SilkS)
+      (effects (font (size 0.5 0.5) (thickness 0.1)))
+    )
