File: saab_bluetooth_aux_kit_v2/saab_bluetooth_aux_kit.sch (KiCad schematic (older format))
At the start: 11 parts, among them J1 Barrel_Jack, U1 MCP1703A-5002_SOT223, U2 ESP32-WROOM-30GPIO, U3 MCP2515-xST, U4 MCP1703A-3302_SOT223, U5 MCP2551-I-P, Y1 Crystal

Commit message: Working on new simplified audio module
Parts:
- removed C1, C2: 27pF, Capacitor_SMD:C_0805_2012Metric_Pad1.15x1.40mm_HandSolder, symbol Device:C_Small
- removed R1, R2: 10k, Resistor_SMD:R_0805_2012Metric_Pad1.15x1.40mm_HandSolder, symbol Device:R_Small
- removed U1: MCP1703A-5002_SOT223, Package_TO_SOT_SMD:SOT-223-3_TabPin2, symbol Regulator_Linear:MCP1703A-5002_SOT223
- removed U2: ESP32-WROOM-30GPIO, custom_footprints:ESP32-WROOM-30GPIO, symbol custom_symbols:ESP32-WROOM-DEVKIT
- removed U3: MCP2515-xST, Package_SO:TSSOP-20_4.4x6.5mm_P0.65mm, symbol Interface_CAN_LIN:MCP2515-xST
- removed U5: MCP2551-I-P, Package_SO:SOIC-8_3.9x4.9mm_P1.27mm, symbol Interface_CAN_LIN:MCP2551-I-SN
- removed Y1: Crystal, Crystal:Crystal_SMD_SeikoEpson_MA505-2Pin_12.7x5.1mm, symbol Device:Crystal
- added U?: PCM5100, Package_SO:TSSOP-20_4.4x6.5mm_P0.65mm, symbol Audio:PCM5100
- added U?: MAX9720, Package_SO:TSSOP-16_4.4x5mm_P0.65mm, symbol custom_symbols:MAX9720
- added U?: ESP32-WROOM-32U, RF_Module:ESP32-WROOM-32U, symbol RF_Module:ESP32-WROOM-32U
Connections:
- new net: U?.1 (GND), U?.15 (GND), U?.38 (GND), U?.39 (GND)
Other:
- note removed: "CAN INTERFACE"
Changed lines of the file:
@@
 $Descr A4 11693 8268
 encoding utf-8
-Sheet 1 2
+Sheet 1 1
 Title ""
 Date ""
@@
 Comment4 ""
 $EndDescr
-$Comp
-L custom_symbols:ESP32-WROOM-DEVKIT U2
-U 1 1 5EA5CF06
-P 5100 4550
-F 0 "U2" H 5075 3282 118 0000 C CNN
-F 1 "ESP32-WROOM-30GPIO" H 5075 3475 118 0000 C CNN
-F 2 "custom_footprints:ESP32-WROOM-30GPIO" H 5100 4550 118 0001 C CNN
-F 3 "" H 5100 4550 118 0001 C CNN
-	1    5100 4550
-	1    0    0    -1
-$EndComp
-Text GLabel 3050 1950 2    50   Input ~ 10
-5VDC
-Text GLabel 2750 2250 2    50   Input ~ 10
-GND
 Text GLabel 4300 5000 0    50   Input ~ 10
 GND
@@
 Text GLabel 5850 5000 2    50   Input ~ 10
 GND
-Text GLabel 8150 1450 0    50   Input ~ 0
-SPI_CS
 Text GLabel 5850 4400 2    50   Input ~ 0
 SPI_CS
-Text GLabel 8150 1550 0    50   Input ~ 0
-SPI_SCLK
 Text GLabel 5850 4300 2    50   Input ~ 0
 SPI_SCLK
-Text GLabel 8150 1350 0    50   Input ~ 0
-SPI_MISO
 Text GLabel 5850 4200 2    50   Input ~ 0
 SPI_MISO
 Text GLabel 5850 3700 2    50   Input ~ 0
-SPI_MOSI
-Text GLabel 8150 1250 0    50   Input ~ 0
 SPI_MOSI
 Text GLabel 4300 4400 0    50   Input ~ 0
@@
 	1    0    0    -1
 $EndComp
-$Comp
-L Regulator_Linear:MCP1703A-5002_SOT223 U1
-U 1 1 5ED69E86
-P 2750 1950
-F 0 "U1" H 2750 2192 50  0000 C CNN
-F 1 "MCP1703A-5002_SOT223" H 2750 2101 50  0000 C CNN
-F 2 "Package_TO_SOT_SMD:SOT-223-3_TabPin2" H 2750 2150 50  0001 C CNN
-F 3 "http://ww1.microchip.com/downloads/en/DeviceDoc/20005122B.pdf" H 2750 1900 50  0001 C CNN
-	1    2750 1950
-	1    0    0    -1
-$EndComp
-$Comp
-L Interface_CAN_LIN:MCP2515-xST U3
-U 1 1 5ED6B86A
-P 8750 1850
-F 0 "U3" H 8750 2831 50  0000 C CNN
-F 1 "MCP2515-xST" H 8750 2740 50  0000 C CNN
-F 2 "Package_SO:TSSOP-20_4.4x6.5mm_P0.65mm" H 8750 950 50  0001 C CIN
-F 3 "http://ww1.microchip.com/downloads/en/DeviceDoc/21801e.pdf" H 8850 1050 50  0001 C CNN
-	1    8750 1850
-	1    0    0    -1
-$EndComp
-$Comp
-L Interface_CAN_LIN:MCP2551-I-SN U5
-U 1 1 5ED6D1AD
-P 10300 1800
-F 0 "U5" H 10300 2381 50  0000 C CNN
-F 1 "MCP2551-I-P" H 10300 2290 50  0000 C CNN
-F 2 "Package_SO:SOIC-8_3.9x4.9mm_P1.27mm" H 10300 1300 50  0001 C CIN
-F 3 "http://ww1.microchip.com/downloads/en/devicedoc/21667d.pdf" H 10300 1800 50  0001 C CNN
-	1    10300 1800
-	1    0    0    -1
-$EndComp
-Text GLabel 8750 2650 2    50   Input ~ 10
-GND
-Text GLabel 10300 2200 2    50   Input ~ 10
-GND
-Text GLabel 8750 1050 2    50   Input ~ 10
-5VDC
-Text GLabel 10300 1400 2    50   Input ~ 10
-5VDC
-Wire Wire Line
-	9350 1250 9600 1250
-Wire Wire Line
-	9600 1250 9600 1700
-Wire Wire Line
-	9600 1700 9800 1700
-Wire Wire Line
-	9800 1600 9550 1600
-Wire Wire Line
-	9550 1600 9550 1350
-Wire Wire Line
-	9550 1350 9350 1350
-$Comp
-L Device:R_Small R2
-U 1 1 5ED6F29E
-P 9800 2250
-F 0 "R2" H 9859 2296 50  0000 L CNN
-F 1 "10k" H 9859 2205 50  0000 L CNN
-F 2 "Resistor_SMD:R_0805_2012Metric_Pad1.15x1.40mm_HandSolder" H 9800 2250 50  0001 C CNN
-F 3 "~" H 9800 2250 50  0001 C CNN
-	1    9800 2250
-	1    0    0    -1
-$EndComp
-Text GLabel 9800 2350 2    50   Input ~ 10
-GND
-Wire Wire Line
-	9800 2150 9800 2000
-$Comp
-L Device:R_Small R1
-U 1 1 5ED769A1
-P 9350 2550
-F 0 "R1" H 9409 2596 50  0000 L CNN
-F 1 "10k" H 9409 2505 50  0000 L CNN
-F 2 "Resistor_SMD:R_0805_2012Metric_Pad1.15x1.40mm_HandSolder" H 9350 2550 50  0001 C CNN
-F 3 "~" H 9350 2550 50  0001 C CNN
-	1    9350 2550
-	1    0    0    -1
-$EndComp
-Text GLabel 9350 2650 2    50   Input ~ 10
-5VDC
-$Comp
-L Device:Crystal Y1
-U 1 1 5ED7BB04
-P 7150 2100
-F 0 "Y1" V 7104 2231 50  0000 L CNN
-F 1 "Crystal" V 7195 2231 50  0000 L CNN
-F 2 "Crystal:Crystal_SMD_SeikoEpson_MA505-2Pin_12.7x5.1mm" H 7150 2100 50  0001 C CNN
-F 3 "~" H 7150 2100 50  0001 C CNN
-	1    7150 2100
-	0    1    1    0
-$EndComp
-$Comp
-L Device:C_Small C2
-U 1 1 5ED7C91E
-P 6850 2250
-F 0 "C2" V 6621 2250 50  0000 C CNN
-F 1 "27pF" V 6712 2250 50  0000 C CNN
-F 2 "Capacitor_SMD:C_0805_2012Metric_Pad1.15x1.40mm_HandSolder" H 6850 2250 50  0001 C CNN
-F 3 "~" H 6850 2250 50  0001 C CNN
-	1    6850 2250
-	0    1    1    0
-$EndComp
-Wire Wire Line
-	6950 1950 7150 1950
-Wire Wire Line
-	7150 2250 6950 2250
-Wire Wire Line
-	6750 1950 6700 1950
-Wire Wire Line
-	6700 1950 6700 2100
-Wire Wire Line
-	6700 2250 6750 2250
-Wire Wire Line
-	6700 2100 6650 2100
-Connection ~ 6700 2100
-Wire Wire Line
-	6700 2100 6700 2250
-Text GLabel 6650 2100 0    50   Input ~ 10
-GND
-Wire Wire Line
-	7450 2050 7450 1950
-Wire Wire Line
-	7450 1950 7150 1950
-Wire Wire Line
-	7450 2050 8150 2050
-Connection ~ 7150 1950
-Wire Wire Line
-	7150 2250 7600 2250
-Wire Wire Line
-	7600 2250 7600 2150
-Wire Wire Line
-	7600 2150 8150 2150
-Connection ~ 7150 2250
-Wire Notes Line
-	6350 750  10900 750
-Wire Notes Line
-	10900 750  10900 2800
-Wire Notes Line
-	10900 2800 6350 2800
-Wire Notes Line
-	6350 2800 6350 750
-Text Notes 6400 850  0    50   ~ 0
-CAN INTERFACE
-$Comp
-L Device:C_Small C1
-U 1 1 5ED7C478
-P 6850 1950
-F 0 "C1" V 6621 1950 50  0000 C CNN
-F 1 "27pF" V 6712 1950 50  0000 C CNN
-F 2 "Capacitor_SMD:C_0805_2012Metric_Pad1.15x1.40mm_HandSolder" H 6850 1950 50  0001 C CNN
-F 3 "~" H 6850 1950 50  0001 C CNN
-	1    6850 1950
-	0    1    1    0
-$EndComp
-$Sheet
-S 7150 3800 1400 1250
-U 5EEA5C0A
-F0 "Sheet5EEA5C09" 50
-F1 "file5EEA5C09.sch" 50
-F2 "VCC" I L 7150 3950 50
-F3 "VDD" I L 7150 3850 50
-F4 "ENABLE" I L 7150 4100 50
-F5 "BCLK" I L 7150 4650 50
-F6 "LRCLK" I L 7150 4550 50
-F7 "OUTP_L" I R 8550 3950 50
-F8 "OUTN_L" I R 8550 4050 50
-F9 "OUTN_R" I R 8550 4900 50
-F10 "OUTP_R" I R 8550 4800 50
-F11 "DIN" I L 7150 4450 50
-$EndSheet
 Text GLabel 7150 4550 0    50   Input ~ 0
 I2S_WSEL
@@
 Text GLabel 2900 1200 2    50   Input ~ 10
 VIN_12V
-Text GLabel 2450 1950 0    50   Input ~ 10
-VIN_12V
 Text GLabel 2450 2650 0    50   Input ~ 10
 VIN_12V
@@
 Text GLabel 7150 4100 0    50   Input ~ 10
 3.3VDC
+$Comp
+L Audio:PCM5100 U?
+U 1 1 5F32AE7E
+P 8650 4100
+F 0 "U?" H 8650 4881 50  0000 C CNN
+F 1 "PCM5100" H 8650 4790 50  0000 C CNN
+F 2 "Package_SO:TSSOP-20_4.4x6.5mm_P0.65mm" H 8600 4850 50  0001 C CNN
+F 3 "http://www.ti.com/lit/ds/symlink/pcm5100.pdf" H 8600 4850 50  0001 C CNN
+	1    8650 4100
+	1    0    0    -1
+$EndComp
+$Comp
+L custom_symbols:MAX9720 U?
+U 1 1 5F331B0A
+P 9950 4100
+F 0 "U?" H 9950 4815 50  0000 C CNN
+F 1 "MAX9720" H 9950 4724 50  0000 C CNN
+F 2 "Package_SO:TSSOP-16_4.4x5mm_P0.65mm" H 9800 4050 50  0001 C CNN
+F 3 "" H 9800 4050 50  0001 C CNN
+	1    9950 4100
+	1    0    0    -1
+$EndComp
+$Comp
+L RF_Module:ESP32-WROOM-32U U?
+U 1 1 5F332B27
+P 5500 1650
+F 0 "U?" H 5500 3231 50  0000 C CNN
+F 1 "ESP32-WROOM-32U" H 5500 3140 50  0000 C CNN
+F 2 "RF_Module:ESP32-WROOM-32U" H 5500 150 50  0001 C CNN
+F 3 "https://www.espressif.com/sites/default/files/documentation/esp32-wroom-32d_esp32-wroom-32u_datasheet_en.pdf" H 5200 1700 50  0001 C CNN
+	1    5500 1650
+	1    0    0    -1
+$EndComp
 $EndSCHEMATC
