File: saab_bluetooth_aux_v3/saab_blue_aux_v3.kicad_pcb (KiCad board)
At the start: 2 copper layers, 60.1 x 60.1 mm, 32 parts, among them J1 Barrel_Jack, J2 USB_B_Micro, J3 Conn_01x08, Q1 BSS138, Q2 BSS138, SW1 SW_EN, SW2 SW_FLASH, U1 PCM5100, U2 MCP1703A-3302_SOT223, U3 MAX9720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

Commit message: Random audio stuff
Parts:
- removed U3: MAX9720, Package_SO:TSSOP-16_4.4x5mm_P0.65mm
- added C1: 10uF, Capacitor_SMD:CP_Elec_4x5.3, F.Cu at (158.9, 82.8)
- added C10: 1uF, Capacitor_SMD:C_0805_2012Metric_Pad1.15x1.40mm_HandSolder, F.Cu at (164.3, 91.8)
- added C11: 100nF, Capacitor_SMD:C_0805_2012Metric_Pad1.15x1.40mm_HandSolder, F.Cu at (154.8, 88.8)
- added C12: 100nF, Capacitor_SMD:C_0805_2012Metric_Pad1.15x1.40mm_HandSolder, F.Cu at (154.8, 91.7)
- added C13: 47uF, Capacitor_SMD:CP_Elec_4x5.3, F.Cu at (158.9, 75.1)
- added C14: 100nF, Capacitor_SMD:C_0805_2012Metric_Pad1.15x1.40mm_HandSolder, F.Cu at (159.6, 88.8)
- added C15: 10uF, Capacitor_SMD:CP_Elec_4x5.3, F.Cu at (164.7, 67.3)
- added C16: 100nF, Capacitor_SMD:C_0805_2012Metric_Pad1.15x1.40mm_HandSolder, F.Cu at (159.6, 91.7)
- added C17: 47uF, Capacitor_SMD:CP_Elec_4x5.3, F.Cu at (164.7, 75.1)
- added C18: 10uF, Capacitor_SMD:CP_Elec_4x5.3, F.Cu at (158.9, 67.3)
- added C8: 10uF, Capacitor_SMD:CP_Elec_4x5.3, F.Cu at (164.7, 82.8)
- added C9: 1uF, Capacitor_SMD:C_0805_2012Metric_Pad1.15x1.40mm_HandSolder, F.Cu at (164.3, 88.9)
- added R1: 10K, Resistor_SMD:R_0805_2012Metric_Pad1.15x1.40mm_HandSolder, F.Cu at (149.2, 90.2)
- J3: value Conn_01x08 -> AudioJack3; footprint Connector_PinHeader_2.54mm:PinHeader_1x08_P2.54mm_Vertical -> Connector_Audio:Jack_3.5mm_CUI_SJ-3523-SMT_Horizontal
- moved J3 52.6 mm to (148.6, 72.4), turned to 0 degrees
- moved D1 29.4 mm to (132.7, 83.2), turned to 90 degrees
- moved J1 24.5 mm to (137.7, 77.3)
- moved U1 7.83 mm to (141.6, 88.3), turned to 270 degrees
- moved U7 6.04 mm to (125.1, 81.6)
- moved C3 6.04 mm to (119.0, 81.7)
- moved I-BUS1 4.32 mm to (126.2, 68.3)
Connections:
- U1 pad 1: (no net) -> VDD_3.3V
- U1 pad 10: (no net) -> Net-(R1-Pad2)
- U1 pad 11: (no net) -> GND
- U1 pad 13: (no net) -> I2S_BCLK
- U1 pad 14: (no net) -> I2S_DIN
- U1 pad 15: (no net) -> I2S_WSEL
- U1 pad 16: (no net) -> GND
- U1 pad 18: (no net) -> Net-(C1-Pad1)
- U1 pad 19: (no net) -> GND
- U1 pad 2: (no net) -> Net-(C18-Pad1)
- U1 pad 20: (no net) -> VDD_3.3V
- U1 pad 3: (no net) -> GND
- U1 pad 4: (no net) -> Net-(C18-Pad2)
- U1 pad 5: (no net) -> Net-(C15-Pad1)
- U1 pad 6: (no net) -> Net-(C10-Pad2)
- U1 pad 7: (no net) -> Net-(C9-Pad2)
- U1 pad 8: (no net) -> VDD_3.3V
- U1 pad 9: (no net) -> GND
- U6 pad 12: Net-(J3-Pad5) -> (no net)
- U6 pad 8: Net-(J3-Pad3) -> (no net)
- U6 pad 9: Net-(J3-Pad4) -> (no net)
