File: saab_bluetooth_aux_v3/saab_blue_aux_v3.sch (KiCad schematic (older format))
At the start: 38 parts, among them J1 Barrel_Jack, J2 USB_B_Micro, J3 Conn_01x08, Q1 BSS138, Q2 BSS138, SW1 SW_EN, SW2 SW_FLASH, U1 PCM5100, U2 MCP1703A-3302_SOT223, U3 MAX9720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

Commit message: Random audio stuff
Parts:
- removed C? (x2): 1uF, Capacitor_SMD:C_0805_2012Metric_Pad1.15x1.40mm_HandSolder, symbol Device:C_Small
- removed J3: Conn_01x08, Connector_PinHeader_2.54mm:PinHeader_1x08_P2.54mm_Vertical, symbol Connector_Generic:Conn_01x08
- removed R?: 10k, Resistor_SMD:R_0805_2012Metric_Pad1.15x1.40mm_HandSolder, symbol Device:R_Small
- removed U3: MAX9720, Package_SO:TSSOP-16_4.4x5mm_P0.65mm, symbol max9720:MAX9720
- added C1, C15, C18, C8: 10uF, Capacitor_SMD:CP_Elec_4x5.3, symbol Device:CP_Small
- added C11, C12, C14, C16: 100nF, Capacitor_SMD:C_0805_2012Metric_Pad1.15x1.40mm_HandSolder, symbol Device:C_Small
- added C13, C17: 47uF, Capacitor_SMD:CP_Elec_4x5.3, symbol Device:CP_Small
- added R1: 10K, Resistor_SMD:R_0805_2012Metric_Pad1.15x1.40mm_HandSolder, symbol Device:R
- J3: renamed from J?; footprint (none) -> Connector_Audio:Jack_3.5mm_CUI_SJ-3523-SMT_Horizontal
- gave numbers to parts that had none: 2
Connections:
- net labels added: GNDD, VDDA
- wire segments 58 -> 65
- no-connect marks 0 -> 1
Other:
- moved on the sheet: C10, C9, J3, U1
