File: hardware/esp32_93NG_btaux_v2/can_interface.kicad_sch (KiCad schematic)
At the start: 4 parts, among them U9 SN65HVD230

Commit message: Adjusted silkscreen labels to reduce clutter. Added GPIO header for external buttons or LEDs. Added second PCB faceplate, for the bottom-side of the assembly.
Other:
- note added: "GMLAN SWCAN terminations. 'Low' is tied to Ground. 'High' is terminated to Ground via 4.7K resistor."
- note added: "SLOPE CONTROL RESISTOR For high-speed operation, this can be replaced with 0Ohms (or bridged with solder)."
Changed lines of the file:
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@@
     (stroke (width 0) (type default) (color 0 0 0 0))
+  )
+  (text "SLOPE CONTROL RESISTOR\nFor high-speed operation, this can be replaced \nwith 0Ohms (or bridged with solder)."
+    (at 106.68 106.68 0)
+    (effects (font (size 1.27 1.27)) (justify right bottom))
+  )
+  (text "GMLAN SWCAN terminations.\n'Low' is tied to Ground.\n'High' is terminated to Ground via 4.7K resistor."
+    (at 154.94 116.84 0)
+    (effects (font (size 1.27 1.27)) (justify left bottom))
   )
   (global_label "CAN_L" (shape input) (at 176.53 95.885 90) (fields_autoplaced)
